File: projects/ESP_DIMMER/ESP8266_Dimmer.brd (EAGLE design)
At the start: 63.5 x 62.5 mm, 39 parts, among them IC1 LD117AS33TR, IC2 TINY24/44/84-SSU, Q1 IRF840

Commit message: Change wrong Diode after first Review
Signed-off-by: Juergen G. Schimmer <schimmi2@gmail.com>
Connections:
- net L: now also D7.A
- net N: no longer D7.A
- net N$2: now also D4.C; no longer D5.C
- net N$3: now also D5.C; no longer D4.C
Changed lines of the file:
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@@
 <setting verticaltext="up"/>
 </settings>
-<grid distance="25" unitdist="mil" unit="mil" style="lines" multiple="4" display="yes" altdistance="0.025" altunitdist="inch" altunit="inch"/>
+<grid distance="0.05" unitdist="inch" unit="inch" style="lines" multiple="2" display="yes" altdistance="0.025" altunitdist="inch" altunit="inch"/>
 <layers>
 <layer number="1" name="Top" color="4" fill="1" visible="yes" active="yes"/>
@@
 <signal name="L">
 <contactref element="D1" pad="C"/>
+<contactref element="R6" pad="2"/>
+<contactref element="D7" pad="A"/>
 <contactref element="D4" pad="A"/>
-<contactref element="R6" pad="2"/>
 <wire x1="10.16" y1="50.8" x2="20.32" y2="55.88" width="0" layer="19" extent="1-1"/>
 <wire x1="10.16" y1="46.99" x2="10.16" y2="50.8" width="0" layer="19" extent="1-1"/>
+<wire x1="10.16" y1="39.37" x2="10.16" y2="46.99" width="0" layer="19" extent="1-1"/>
 </signal>
 <signal name="N">
 <contactref element="D2" pad="C"/>
 <contactref element="D5" pad="A"/>
-<contactref element="D7" pad="A"/>
-<wire x1="10.16" y1="31.75" x2="10.16" y2="39.37" width="0" layer="19" extent="1-1"/>
 <wire x1="10.16" y1="12.7" x2="10.16" y2="31.75" width="0" layer="19" extent="1-1"/>
 </signal>
@@
 </signal>
 <signal name="N$2">
-<contactref element="D5" pad="C"/>
 <contactref element="D6" pad="C"/>
 <contactref element="Q1" pad="2"/>
 <contactref element="R9" pad="2"/>
-<wire x1="25.4" y1="31.75" x2="29.21" y2="31.75" width="0" layer="19" extent="1-1"/>
-<wire x1="25.4" y1="25.4" x2="25.4" y2="31.75" width="0" layer="19" extent="1-1"/>
-<wire x1="30.48" y1="25.4" x2="25.4" y2="25.4" width="0" layer="19" extent="1-1"/>
+<contactref element="D4" pad="C"/>
+<wire x1="29.21" y1="31.75" x2="20.32" y2="46.99" width="0" layer="19" extent="1-1"/>
+<wire x1="30.48" y1="25.4" x2="29.21" y2="31.75" width="0" layer="19" extent="1-1"/>
+<wire x1="25.4" y1="25.4" x2="30.48" y2="25.4" width="0" layer="19" extent="1-1"/>
 </signal>
 <signal name="N$3">
-<contactref element="D4" pad="C"/>
 <contactref element="D8" pad="C"/>
+<contactref element="R2" pad="1"/>
 <contactref element="D7" pad="C"/>
-<contactref element="R2" pad="1"/>
-<wire x1="20.32" y1="43.18" x2="20.32" y2="46.99" width="0" layer="19" extent="1-1"/>
+<contactref element="D5" pad="C"/>
 <wire x1="20.32" y1="39.37" x2="20.32" y2="43.18" width="0" layer="19" extent="1-1"/>
 <wire x1="22.86" y1="39.37" x2="20.32" y2="39.37" width="0" layer="19" extent="1-1"/>
+<wire x1="25.4" y1="31.75" x2="22.86" y2="39.37" width="0" layer="19" extent="1-1"/>
 </signal>
 <signal name="N$6">
